Commit message: Fix xacro formats

File: chapter6/fourth_robot_description/robots/fourth_robot.urdf.xacro (robot description, xacro)
@@ -66,5 +66,5 @@
   <xacro:wheel_gazebo_v0 prefix="right"/>
   <xacro:wheel_gazebo_v0 prefix="left"/>
-  <xacro:wheel_gazebo_control_v0 rate="25"/>
+  <!--xacro:wheel_gazebo_control_v0 rate="25"/-->
   <!-- LRF -->
   <xacro:lrf_gazebo_v0 prefix="front"

File: chapter6/fourth_robot_description/urdf/base/base.urdf.xacro (robot description, xacro)
@@ -4,5 +4,5 @@
   <xacro:macro name="base_v0" params="parent *joint_origin">
 	<joint name="base_link_joint" type="fixed">
-	  <insert_block name="joint_origin"/>
+	  <xacro:insert_block name="joint_origin"/>
 	  <parent link="${parent}"/>
 	  <child link="base_link"/>

File: chapter6/fourth_robot_description/urdf/wheel/wheel.urdf.xacro (robot description, xacro)
@@ -4,13 +4,13 @@
   <xacro:include filename="$(find fourth_robot_description)/urdf/wheel/wheel.transmission.xacro"/>
   <xacro:include filename="$(find fourth_robot_description)/urdf/wheel/wheel.gazebo.xacro"/>
-  <property name="wheel_radius" value="0.20316"/>
-  <property name="wheel_length" value="0.032"/>
-  <property name="wheel_mass" value="2.0"/>
+  <xacro:property name="wheel_radius" value="0.20316"/>
+  <xacro:property name="wheel_length" value="0.032"/>
+  <xacro:property name="wheel_mass" value="2.0"/>
   <xacro:macro name="wheel_v0" params="prefix parent *joint_origin *joint_axis">
 	<joint name="${prefix}_wheel_joint" type="continuous">
-	  <insert_block name="joint_origin"/>
+	  <xacro:insert_block name="joint_origin"/>
 	  <parent link="${parent}"/>
 	  <child link="${prefix}_wheel_link"/>
-	  <insert_block name="joint_axis"/>
+	  <xacro:insert_block name="joint_axis"/>
 	</joint>
 	<link name="${prefix}_wheel_link">
